Commit message: add controller run scripts

File: urdf/kr210.urdf.xacro (robot description, xacro)
@@ -1,4 +1,4 @@
 <?xml version="1.0"?>
-<robot name="kuka_kr210_arm" xmlns:xacro="http://www.ros.org/wiki/xacro">
+<robot name="kr210_kuka_manipulator" xmlns:xacro="http://www.ros.org/wiki/xacro">
 <!-- pan_tilt.xacro inorder > pan_tilt_generated.urdf -->
   <!--Define constants-->
@@ -17,5 +17,5 @@
   <xacro:property name="vacuum_gripper_radius" value="0.1" />
   <!--Import gazebo elements-->
-  <xacro:include filename="$(find kuka_kr210_arm)/urdf/kr210.gazebo.xacro" />
+  <xacro:include filename="$(find kr210_kuka_manipulator)/urdf/kr210.gazebo.xacro" />
   <!--Links-->
   <link name="base_footprint"/>
@@ -29,14 +29,14 @@
       <origin xyz="0 0 0" rpy="${-pi/2} 0 0"/>
       <geometry>
-        <mesh filename="package://kuka_kr210_arm/meshes/visual/base_link.dae"/>
-      </geometry>
-      <material name="">
-        <color rgba="0.75294 0.75294 0.75294 1"/>
-      </material>
-    </visual>
-    <collision>
-      <origin xyz="0 0 0" rpy="${-pi/2} 0 0"/>
-      <geometry>
-        <mesh filename="package://kuka_kr210_arm/meshes/collision/base_link.stl"/>
+        <mesh filename="package://kr210_kuka_manipulator/meshes/visual/base_link.dae"/>
+      </geometry>
+      <material name="">
+        <color rgba="0.75294 0.75294 0.75294 1"/>
+      </material>
+    </visual>
+    <collision>
+      <origin xyz="0 0 0" rpy="${-pi/2} 0 0"/>
+      <geometry>
+        <mesh filename="package://kr210_kuka_manipulator/meshes/collision/base_link.stl"/>
       </geometry>
     </collision>
@@ -51,14 +51,14 @@
       <origin xyz="0 0 0" rpy="0 0 0"/>
       <geometry>
-        <mesh filename="package://kuka_kr210_arm/meshes/visual/link_1.dae"/>
-      </geometry>
-      <material name="">
-        <color rgba="0.75294 0.75294 0.75294 1"/>
-      </material>
-    </visual>
-    <collision>
-      <origin xyz="0 0 0" rpy="0 0 0"/>
-      <geometry>
-        <mesh filename="package://kuka_kr210_arm/meshes/collision/link_1.stl"/>
+        <mesh filename="package://kr210_kuka_manipulator/meshes/visual/link_1.dae"/>
+      </geometry>
+      <material name="">
+        <color rgba="0.75294 0.75294 0.75294 1"/>
+      </material>
+    </visual>
+    <collision>
+      <origin xyz="0 0 0" rpy="0 0 0"/>
+      <geometry>
+        <mesh filename="package://kr210_kuka_manipulator/meshes/collision/link_1.stl"/>
       </geometry>
     </collision>
@@ -73,14 +73,14 @@
       <origin xyz="0 0 0" rpy="${-pi/2} 0 0"/>
       <geometry>
-        <mesh filename="package://kuka_kr210_arm/meshes/visual/link_2.dae"/>
-      </geometry>
-      <material name="">
-        <color rgba="0.75294 0.75294 0.75294 1"/>
-      </material>
-    </visual>
-    <collision>
-      <origin xyz="0 0 0" rpy="0 0 0"/>
-      <geometry>
-        <mesh filename="package://kuka_kr210_arm/meshes/collision/link_2.stl"/>
+        <mesh filename="package://kr210_kuka_manipulator/meshes/visual/link_2.dae"/>
+      </geometry>
+      <material name="">
+        <color rgba="0.75294 0.75294 0.75294 1"/>
+      </material>
+    </visual>
+    <collision>
+      <origin xyz="0 0 0" rpy="0 0 0"/>
+      <geometry>
+        <mesh filename="package://kr210_kuka_manipulator/meshes/collision/link_2.stl"/>
       </geometry>
     </collision>
@@ -95,5 +95,5 @@
       <origin xyz="0 -0.184 0" rpy="${-pi/2} 0 0"/>
       <geometry>
-        <mesh filename="package://kuka_kr210_arm/meshes/visual/link_3.dae"/>
+        <mesh filename="package://kr210_kuka_manipulator/meshes/visual/link_3.dae"/>
       </geometry>
       <material name="">
@@ -104,5 +104,5 @@
       <origin xyz="0 -0.184 0" rpy="0 0 0"/>
       <geometry>
-        <mesh filename="package://kuka_kr210_arm/meshes/collision/link_3.stl"/>
+        <mesh filename="package://kr210_kuka_manipulator/meshes/collision/link_3.stl"/>
       </geometry>
     </collision>
@@ -117,14 +117,14 @@
       <origin xyz="0 0 0" rpy="${-pi/2} 0 0"/>
       <geometry>
-        <mesh filename="package://kuka_kr210_arm/meshes/visual/link_4.dae"/>
-      </geometry>
-      <material name="">
-        <color rgba="0.75294 0.75294 0.75294 1"/>
-      </material>
-    </visual>
-    <collision>
-      <origin xyz="0 0 0" rpy="0 0 0"/>
-      <geometry>
-        <mesh filename="package://kuka_kr210_arm/meshes/collision/link_4.stl"/>
+        <mesh filename="package://kr210_kuka_manipulator/meshes/visual/link_4.dae"/>
+      </geometry>
+      <material name="">
+        <color rgba="0.75294 0.75294 0.75294 1"/>
+      </material>
+    </visual>
+    <collision>
+      <origin xyz="0 0 0" rpy="0 0 0"/>
+      <geometry>
+        <mesh filename="package://kr210_kuka_manipulator/meshes/collision/link_4.stl"/>
       </geometry>
     </collision>
@@ -139,14 +139,14 @@
       <origin xyz="0 0 0" rpy="${-pi/2} 0 0"/>
       <geometry>
-        <mesh filename="package://kuka_kr210_arm/meshes/visual/link_5.dae"/>
-      </geometry>
-      <material name="">
-        <color rgba="0.75294 0.75294 0.75294 1"/>
-      </material>
-    </visual>
-    <collision>
-      <origin xyz="0 0 0" rpy="0 0 0"/>
-      <geometry>
-        <mesh filename="package://kuka_kr210_arm/meshes/collision/link_5.stl"/>
+        <mesh filename="package://kr210_kuka_manipulator/meshes/visual/link_5.dae"/>
+      </geometry>
+      <material name="">
+        <color rgba="0.75294 0.75294 0.75294 1"/>
+      </material>
+    </visual>
+    <collision>
+      <origin xyz="0 0 0" rpy="0 0 0"/>
+      <geometry>
+        <mesh filename="package://kr210_kuka_manipulator/meshes/collision/link_5.stl"/>
       </geometry>
     </collision>
@@ -161,14 +161,14 @@
       <origin xyz="0 0 0" rpy="0 0 0"/>
       <geometry>
-        <mesh filename="package://kuka_kr210_arm/meshes/visual/link_6.dae"/>
-      </geometry>
-      <material name="">
-        <color rgba="0.75294 0.75294 0.75294 1"/>
-      </material>
-    </visual>
-    <collision>
-      <origin xyz="0 0 0" rpy="0 0 0"/>
-      <geometry>
-        <mesh filename="package://kuka_kr210_arm/meshes/collision/link_6.stl"/>
+        <mesh filename="package://kr210_kuka_manipulator/meshes/visual/link_6.dae"/>
+      </geometry>
+      <material name="">
+        <color rgba="0.75294 0.75294 0.75294 1"/>
+      </material>
+    </visual>
+    <collision>
+      <origin xyz="0 0 0" rpy="0 0 0"/>
+      <geometry>
+        <mesh filename="package://kr210_kuka_manipulator/meshes/collision/link_6.stl"/>
       </geometry>
     </collision>
@@ -213,11 +213,11 @@
       <origin xyz="0 0 0" rpy="0 0 0"/>
       <geometry>
-        <mesh filename="package://kuka_kr210_arm/meshes/visual/gripper_base.dae"/>
-      </geometry>
-    </visual>
-    <collision>
-      <origin xyz="0 0 0" rpy="0 0 0"/>
-      <geometry>
-        <mesh filename="package://kuka_kr210_arm/meshes/visual/gripper_base.dae"/>
+        <mesh filename="package://kr210_kuka_manipulator/meshes/visual/gripper_base.dae"/>
+      </geometry>
+    </visual>
+    <collision>
+      <origin xyz="0 0 0" rpy="0 0 0"/>
+      <geometry>
+        <mesh filename="package://kr210_kuka_manipulator/meshes/visual/gripper_base.dae"/>
       </geometry>
     </collision>
@@ -232,11 +232,11 @@
       <origin xyz="0 0 0" rpy="0 0 0"/>
       <geometry>
-        <mesh filename="package://kuka_kr210_arm/meshes/visual/finger_right.dae"/>
-      </geometry>
-    </visual>
-    <collision>
-      <origin xyz="0 0 0" rpy="0 0 0"/>
-      <geometry>
-        <mesh filename="package://kuka_kr210_arm/meshes/collision/finger_right_collision.dae"/>
+        <mesh filename="package://kr210_kuka_manipulator/meshes/visual/finger_right.dae"/>
+      </geometry>
+    </visual>
+    <collision>
+      <origin xyz="0 0 0" rpy="0 0 0"/>
+      <geometry>
+        <mesh filename="package://kr210_kuka_manipulator/meshes/collision/finger_right_collision.dae"/>
       </geometry>
     </collision>
@@ -251,11 +251,11 @@
       <origin xyz="0 0 0" rpy="0 0 0"/>
       <geometry>
-        <mesh filename="package://kuka_kr210_arm/meshes/visual/finger_left.dae"/>
-      </geometry>
-    </visual>
-    <collision>
-      <origin xyz="0 0 0" rpy="0 0 0"/>
-      <geometry>
-        <mesh filename="package://kuka_kr210_arm/meshes/collision/finger_left_collision.dae"/>
+        <mesh filename="package://kr210_kuka_manipulator/meshes/visual/finger_left.dae"/>
+      </geometry>
+    </visual>
+    <collision>
+      <origin xyz="0 0 0" rpy="0 0 0"/>
+      <geometry>
+        <mesh filename="package://kr210_kuka_manipulator/meshes/collision/finger_left_collision.dae"/>
       </geometry>
     </collision>

File: urdf/kr210_gazebo.urdf (robot description, URDF)
Before this commit: robot kuka_kr210_arm, 11 links, 10 joints
Links:
- link base_link: geometry collision mesh filename=package://kr210_kuka_manipulator/meshes/collision/base_link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; visual mesh filename=package://kr210_kuka_manipulator/meshes/visual/base_link.dae
- link gripper_link: geometry collision mesh filename=package://kr210_kuka_manipulator/meshes/visual/gripper_base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; visual mesh filename=package://kr210_kuka_manipulator/meshes/visual/gripper_base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
- link left_gripper_finger_link: geometry collision mesh filename=package://kr210_kuka_manipulator/meshes/collision/finger_le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; visual mesh filename=package://kr210_kuka_manipulator/meshes/visual/finger_left.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
- link link_1: geometry collision mesh filename=package://kr210_kuka_manipulator/meshes/collision/link_1.stl; visual mesh filename=package://kr210_kuka_manipulator/meshes/visual/link_1.dae
- link link_2: geometry collision mesh filename=package://kr210_kuka_manipulator/meshes/collision/link_2.stl; visual mesh filename=package://kr210_kuka_manipulator/meshes/visual/link_2.dae
- link link_3: geometry collision mesh filename=package://kr210_kuka_manipulator/meshes/collision/link_3.stl; visual mesh filename=package://kr210_kuka_manipulator/meshes/visual/link_3.dae
- link link_4: geometry collision mesh filename=package://kr210_kuka_manipulator/meshes/collision/link_4.stl; visual mesh filename=package://kr210_kuka_manipulator/meshes/visual/link_4.dae
- link link_5: geometry collision mesh filename=package://kr210_kuka_manipulator/meshes/collision/link_5.stl; visual mesh filename=package://kr210_kuka_manipulator/meshes/visual/link_5.dae
- link link_6: geometry collision mesh filename=package://kr210_kuka_manipulator/meshes/collision/link_6.stl; visual mesh filename=package://kr210_kuka_manipulator/meshes/visual/link_6.dae
- link right_gripper_finger_link: geometry collision mesh filename=package://kr210_kuka_manipulator/meshes/collision/finger_ri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; visual mesh filename=package://kr210_kuka_manipulator/meshes/visual/finger_right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
